Commit message: torso limits changed

File: cob_description/urdf/cob3_torso/torso_v2.urdf.xacro (robot description, xacro)
@@ -25,6 +25,6 @@
       <dynamics damping="25.0" friction="10.0"/>
       <calibration rising="${torso_lower_neck_tilt_ref}"/>
-      <limit effort="200.0" lower="-0.25" upper="0.21" velocity="0.5"/>
-      <!--safety_controller k_position="20" k_velocity="50" soft_lower_limit="${-0.25 + 0.01}" soft_upper_limit="${0.25 - 0.01}" /-->
+      <limit effort="200.0" lower="-0.37" upper="0.11" velocity="0.5"/>
+      <!--safety_controller k_position="20" k_velocity="50" soft_lower_limit="${-0.37 + 0.01}" soft_upper_limit="${0.11 - 0.01}" /-->
     </joint>
     <link name="${name}_lower_neck_tilt_link">
@@ -56,6 +56,6 @@
       <dynamics damping="25.0" friction="10.0"/>
       <calibration rising="${torso_pan_ref}"/>
-      <limit effort="200.0" lower="-0.12" upper="0.12" velocity="0.5"/>
-      <!--safety_controller k_position="20" k_velocity="50" soft_lower_limit="${-0.2 + 0.01}" soft_upper_limit="${0.2 - 0.01}" /-->
+      <limit effort="200.0" lower="-0.18" upper="0.18" velocity="0.5"/>
+      <!--safety_controller k_position="20" k_velocity="50" soft_lower_limit="${-0.18 + 0.01}" soft_upper_limit="${0.18 - 0.01}" /-->
     </joint>
     <link name="${name}_pan_link">
@@ -74,6 +74,6 @@
       <dynamics damping="25.0" friction="10.0"/>
       <calibration rising="${torso_upper_neck_tilt_ref}"/>
-      <limit effort="200.0" lower="-0.37" upper="0.37" velocity="0.5"/>
-      <!--safety_controller k_position="20" k_velocity="50" soft_lower_limit="${-0.4 + 0.01}" soft_upper_limit="${0.4 - 0.01}" /-->
+      <limit effort="200.0" lower="-0.4" upper="0.39" velocity="0.5"/>
+      <!--safety_controller k_position="20" k_velocity="50" soft_lower_limit="${-0.4 + 0.01}" soft_upper_limit="${0.39 - 0.01}" /-->
     </joint>
     <link name="${name}_upper_neck_tilt_link">

File: cob_description/urdf/sensors/kinect.urdf.xacro (robot description, xacro)
@@ -13,5 +13,5 @@
       </xacro:box_inertial>
       <visual>
-        <origin xyz="0 0 -0.03" rpy="0 0 0" />
+        <origin xyz="0 0 0.0" rpy="0 0 0" />
         <geometry>
           <box size="0.02 0.02 0.02"/>
@@ -20,5 +20,5 @@
       </visual>
       <collision>
-        <origin xyz="0 0 -0.03" rpy="0 0 0" />
+        <origin xyz="0 0 0.0" rpy="0 0 0" />
         <geometry>
            <box size="0.02 0.02 0.02"/>
