Commit message: Drehrichtung der Torso Gelenke geändert

File: cob_description/urdf/cob3_torso/torso_dai.urdf.xacro (robot description, xacro)
@@ -35,5 +35,5 @@
       <parent link="${name}_base_link"/>
       <child link="${name}_lower_neck_tilt_link"/>
-      <axis xyz="0 1 0" />
+      <axis xyz="0 -1 0" />
       <dynamics damping="25.0" friction="10.0"/>
       <calibration rising="${torso_lower_neck_tilt_ref}"/>
@@ -66,5 +66,5 @@
       <parent link="${name}_lower_neck_tilt_link"/>
       <child link="${name}_pan_link"/>
-      <axis xyz="0 1 0" />
+      <axis xyz="0 -1 0" />
       <dynamics damping="25.0" friction="10.0"/>
       <calibration rising="${torso_pan_ref}"/>

Commit message: torso model: rotation around z axis

File: cob_description/urdf/cob3_torso/torso_dai.urdf.xacro (robot description, xacro)
@@ -17,5 +17,5 @@
       </inertial>
       <visual>
-        <origin xyz="0 0 0" rpy="0 0 ${-M_PI/2}" />
+        <origin xyz="0 0 0" rpy="${-M_PI/2} ${-M_PI/2} 0" />
         <geometry>
           <mesh filename="package://cob_description/meshes/cob3_torso/torso_base_high.dae" scale="0.01 0.01 0.01"/>
@@ -24,5 +24,5 @@
       </visual>
       <collision>
-        <origin xyz="0 0 0" rpy="0 0 ${-M_PI/2}" />
+        <origin xyz="0 0 0" rpy="${-M_PI/2} ${-M_PI/2} 0" />
         <geometry>
           <mesh filename="package://cob_description/meshes/cob3_torso/torso_base_low.dae" scale="0.01 0.01 0.01"/>
@@ -32,21 +32,21 @@
     <!-- joint between base_link and torso_lower_neck_tilt_link -->
     <joint name="${name}_lower_neck_tilt_joint" type="revolute">
-      <origin xyz="0 0 0.08" rpy="0 0 0" />
+      <origin xyz="0 0.08 0" rpy="0 0 0" />
       <parent link="${name}_base_link"/>
       <child link="${name}_lower_neck_tilt_link"/>
-      <axis xyz="0 -1 0" />
+      <axis xyz="0 0 1" />
       <dynamics damping="25.0" friction="10.0"/>
       <calibration rising="${torso_lower_neck_tilt_ref}"/>
-      <limit effort="200.0" lower="-0.9" upper="0.9" velocity="0.5"/>
+      <limit effort="200.0" lower="-0.5" upper="0.5" velocity="0.5"/>
       <!--safety_controller k_position="20" k_velocity="50" soft_lower_limit="${-0.37 + 0.01}" soft_upper_limit="${0.11 - 0.01}" /-->
     </joint>
     <link name="${name}_lower_neck_tilt_link">
       <inertial>
-        <origin xyz="0 0 -0.055" rpy="0 0 0"/>
-        <mass value="0.2"/>
-        <inertia ixx="1" ixy="0" ixz="0" iyy="1" iyz="0" izz="1" />
+        <origin xyz="0 0 0" rpy="0 0 0"/>
+        <mass value="6.209720"/>
+        <inertia ixx="0.171118" ixy="0.002544" ixz="-0.000000" iyy="0.083077" iyz="0.000000" izz="0.120948" />
       </inertial>
       <visual>
-        <origin xyz="0 -0.055 0" rpy="0 0 0" />
+        <origin xyz="0 0 0.055" rpy="${-M_PI/2} 0 0" />
         <geometry>
           <mesh filename="package://cob_description/meshes/cob3_torso/torso_tilt_high.dae" scale="0.01 0.01 0.01"/>
@@ -55,5 +55,5 @@
       </visual>
       <collision>
-        <origin xyz="0 -0.055 0" rpy="0 0 0" />
+        <origin xyz="0 0 0.055" rpy="${-M_PI/2} 0 0" />
         <geometry>
           <mesh filename="package://cob_description/meshes/cob3_torso/torso_tilt_low.dae" scale="0.01 0.01 0.01"/>
@@ -63,8 +63,8 @@
     <!-- joint between torso_lower_neck_tilt_link and torso_pan_link -->
     <joint name="${name}_pan_joint" type="revolute">
-      <origin xyz="0 0 0.0715" rpy="${M_PI/2} 0 0" />
+      <origin xyz="0 0 0" rpy="${M_PI/2} 0 0" />
       <parent link="${name}_lower_neck_tilt_link"/>
       <child link="${name}_pan_link"/>
-      <axis xyz="0 -1 0" />
+      <axis xyz="0 0 1" />
       <dynamics damping="25.0" friction="10.0"/>
       <calibration rising="${torso_pan_ref}"/>
@@ -79,5 +79,5 @@
       </inertial>
       <visual>
-        <origin xyz="0 0 0" rpy="0 0 0" />
+        <origin xyz="0 0 -0.0715" rpy="${-M_PI/2} 0 ${M_PI}" />
         <geometry>
           <mesh filename="package://cob_description/meshes/cob3_torso/torso_pan_high.dae" scale="0.01 0.01 0.01"/>
@@ -86,5 +86,5 @@
       </visual>
       <collision>
-        <origin xyz="0 0 0" rpy="0 0 0" />
+        <origin xyz="0 0 -0.0715" rpy="${-M_PI/2} 0 ${M_PI}" />
         <geometry>
           <mesh filename="package://cob_description/meshes/cob3_torso/torso_pan_low.dae" scale="0.01 0.01 0.01"/>
@@ -94,5 +94,5 @@
     <!-- joint between torso_pan_link and torso_upper_neck_tilt_link -->
     <joint name="${name}_upper_neck_tilt_joint" type="revolute">
-      <origin xyz="0 0.185 0" rpy="0 0 0" />
+      <origin xyz="0 0 -0.2565" rpy="-${M_PI/2} 0 0" />
       <parent link="${name}_pan_link"/>
       <child link="${name}_upper_neck_tilt_link"/>
@@ -105,10 +105,10 @@
     <link name="${name}_upper_neck_tilt_link">
       <inertial>
-        <origin xyz="0 0 -0.055" rpy="0 0 0"/>
+        <origin xyz="0 0 0" rpy="0 0 0"/>
         <mass value="6.744238"/>
         <inertia ixx="0.01" ixy="0" ixz="0" iyy="0.01" iyz="0" izz="0.01" />
       </inertial>
       <visual>
-        <origin xyz="0 0 -0.055" rpy="-${M_PI/2} ${M_PI} 0" />
+        <origin xyz="0 0 0.055" rpy="-${M_PI/2} 0 0" />
         <geometry>
           <mesh filename="package://cob_description/meshes/cob3_torso/torso_tilt_high.dae" scale="0.01 0.01 0.01"/>
@@ -117,5 +117,5 @@
       </visual>
       <collision>
-        <origin xyz="0 0 -0.055" rpy="-${M_PI/2} ${M_PI} 0" />
+        <origin xyz="0 0 0.055" rpy="-${M_PI/2} 0 0" />
         <geometry>
           <!--mesh filename="package://cob_description/meshes/cob3_torso/upper_neck_collision.stl" /-->

Commit message: new limits for torso (hardware limits changed)

File: cob_description/urdf/cob3_torso/torso_dai.urdf.xacro (robot description, xacro)
@@ -38,5 +38,5 @@
       <dynamics damping="25.0" friction="10.0"/>
       <calibration rising="${torso_lower_neck_tilt_ref}"/>
-      <limit effort="200.0" lower="-0.5" upper="0.5" velocity="0.5"/>
+      <limit effort="200.0" lower="-0.43" upper="0.43" velocity="0.5"/>
       <!--safety_controller k_position="20" k_velocity="50" soft_lower_limit="${-0.37 + 0.01}" soft_upper_limit="${0.11 - 0.01}" /-->
     </joint>
@@ -69,5 +69,5 @@
       <dynamics damping="25.0" friction="10.0"/>
       <calibration rising="${torso_pan_ref}"/>
-      <limit effort="200.0" lower="-1.5" upper="1.5" velocity="0.5"/>
+      <limit effort="200.0" lower="-1.57" upper="1.57" velocity="0.5"/>
       <!--safety_controller k_position="20" k_velocity="50" soft_lower_limit="${-0.18 + 0.01}" soft_upper_limit="${0.18 - 0.01}" /-->
     </joint>
@@ -100,5 +100,5 @@
       <dynamics damping="25.0" friction="10.0"/>
       <calibration rising="${torso_upper_neck_tilt_ref}"/>
-      <limit effort="200.0" lower="-0.9" upper="0.9" velocity="0.5"/>
+      <limit effort="200.0" lower="-0.78" upper="0.78" velocity="0.5"/>
       <!--safety_controller k_position="20" k_velocity="50" soft_lower_limit="${-0.4 + 0.01}" soft_upper_limit="${0.39 - 0.01}" /-->
     </joint>

Commit message: changed color of torso

File: cob_description/urdf/cob3_torso/torso_dai.urdf.xacro (robot description, xacro)
@@ -21,5 +21,5 @@
           <mesh filename="package://cob_description/meshes/cob3_torso/torso_base_high.dae" scale="0.01 0.01 0.01"/>
         </geometry>
-        <material name="IPA/LightGrey" />
+        <material name="IPA/Metal" />
       </visual>
       <collision>
@@ -52,5 +52,5 @@
           <mesh filename="package://cob_description/meshes/cob3_torso/torso_tilt_high.dae" scale="0.01 0.01 0.01"/>
         </geometry>
-        <material name="IPA/LightGrey" />
+        <material name="IPA/Metal" />
       </visual>
       <collision>
@@ -83,5 +83,5 @@
           <mesh filename="package://cob_description/meshes/cob3_torso/torso_pan_high.dae" scale="0.01 0.01 0.01"/>
         </geometry>
-        <material name="IPA/LightGrey" />
+        <material name="IPA/Metal" />
       </visual>
       <collision>
@@ -114,5 +114,5 @@
           <mesh filename="package://cob_description/meshes/cob3_torso/torso_tilt_high.dae" scale="0.01 0.01 0.01"/>
         </geometry>
-        <material name="IPA/LightGrey" />
+        <material name="IPA/Metal" />
       </visual>
       <collision>
@@ -141,5 +141,5 @@
           <mesh filename="package://cob_description/meshes/cob3_torso/head_base.dae" scale="0.01 0.01 0.01"/>
         </geometry>
-        <material name="IPA/LightGrey" />
+        <material name="IPA/Metal" />
       </visual>
       <collision>

Commit message: lower torso velocity limits

File: cob_description/urdf/cob3_torso/torso_dai.urdf.xacro (robot description, xacro)
@@ -38,5 +38,5 @@
       <dynamics damping="25.0" friction="10.0"/>
       <calibration rising="${torso_lower_neck_tilt_ref}"/>
-      <limit effort="200.0" lower="-0.43" upper="0.43" velocity="0.5"/>
+      <limit effort="200.0" lower="-0.43" upper="0.43" velocity="0.4"/>
       <!--safety_controller k_position="20" k_velocity="50" soft_lower_limit="${-0.37 + 0.01}" soft_upper_limit="${0.11 - 0.01}" /-->
     </joint>
@@ -69,5 +69,5 @@
       <dynamics damping="25.0" friction="10.0"/>
       <calibration rising="${torso_pan_ref}"/>
-      <limit effort="200.0" lower="-1.57" upper="1.57" velocity="0.5"/>
+      <limit effort="200.0" lower="-1.57" upper="1.57" velocity="0.4"/>
       <!--safety_controller k_position="20" k_velocity="50" soft_lower_limit="${-0.18 + 0.01}" soft_upper_limit="${0.18 - 0.01}" /-->
     </joint>
@@ -100,5 +100,5 @@
       <dynamics damping="25.0" friction="10.0"/>
       <calibration rising="${torso_upper_neck_tilt_ref}"/>
-      <limit effort="200.0" lower="-0.78" upper="0.78" velocity="0.5"/>
+      <limit effort="200.0" lower="-0.78" upper="0.78" velocity="0.4"/>
       <!--safety_controller k_position="20" k_velocity="50" soft_lower_limit="${-0.4 + 0.01}" soft_upper_limit="${0.39 - 0.01}" /-->
     </joint>

Commit message: torso color

File: cob_description/urdf/cob3_torso/torso_dai.urdf.xacro (robot description, xacro)
@@ -21,5 +21,5 @@
           <mesh filename="package://cob_description/meshes/cob3_torso/torso_base_high.dae" scale="0.01 0.01 0.01"/>
         </geometry>
-        <material name="IPA/Metal" />
+        <material name="Schunk/LightGrey" />
       </visual>
       <collision>
@@ -52,5 +52,5 @@
           <mesh filename="package://cob_description/meshes/cob3_torso/torso_tilt_high.dae" scale="0.01 0.01 0.01"/>
         </geometry>
-        <material name="IPA/Metal" />
+        <material name="Schunk/LightGrey" />
       </visual>
       <collision>
@@ -83,5 +83,5 @@
           <mesh filename="package://cob_description/meshes/cob3_torso/torso_pan_high.dae" scale="0.01 0.01 0.01"/>
         </geometry>
-        <material name="IPA/Metal" />
+        <material name="Schunk/LightGrey" />
       </visual>
       <collision>
@@ -114,5 +114,5 @@
           <mesh filename="package://cob_description/meshes/cob3_torso/torso_tilt_high.dae" scale="0.01 0.01 0.01"/>
         </geometry>
-        <material name="IPA/Metal" />
+        <material name="Schunk/LightGrey" />
       </visual>
       <collision>
@@ -141,5 +141,5 @@
           <mesh filename="package://cob_description/meshes/cob3_torso/head_base.dae" scale="0.01 0.01 0.01"/>
         </geometry>
-        <material name="IPA/Metal" />
+        <material name="Schunk/LightGrey" />
       </visual>
       <collision>

Commit message: torso limits

File: cob_description/urdf/cob3_torso/torso_dai.urdf.xacro (robot description, xacro)
@@ -38,5 +38,5 @@
       <dynamics damping="25.0" friction="10.0"/>
       <calibration rising="${torso_lower_neck_tilt_ref}"/>
-      <limit effort="200.0" lower="-0.43" upper="0.43" velocity="0.4"/>
+      <limit effort="200.0" lower="-0.43" upper="0.78" velocity="0.4"/>
       <!--safety_controller k_position="20" k_velocity="50" soft_lower_limit="${-0.37 + 0.01}" soft_upper_limit="${0.11 - 0.01}" /-->
     </joint>
@@ -69,5 +69,5 @@
       <dynamics damping="25.0" friction="10.0"/>
       <calibration rising="${torso_pan_ref}"/>
-      <limit effort="200.0" lower="-1.57" upper="1.57" velocity="0.4"/>
+      <limit effort="200.0" lower="-1.65" upper="1.65" velocity="0.4"/>
       <!--safety_controller k_position="20" k_velocity="50" soft_lower_limit="${-0.18 + 0.01}" soft_upper_limit="${0.18 - 0.01}" /-->
     </joint>
@@ -100,5 +100,5 @@
       <dynamics damping="25.0" friction="10.0"/>
       <calibration rising="${torso_upper_neck_tilt_ref}"/>
-      <limit effort="200.0" lower="-0.78" upper="0.78" velocity="0.4"/>
+      <limit effort="200.0" lower="-1.12" upper="0.78" velocity="0.4"/>
       <!--safety_controller k_position="20" k_velocity="50" soft_lower_limit="${-0.4 + 0.01}" soft_upper_limit="${0.39 - 0.01}" /-->
     </joint>

Commit message: new head collision model

File: cob_description/urdf/cob3_torso/torso_dai.urdf.xacro (robot description, xacro)
@@ -146,5 +146,5 @@
         <origin xyz="0 0 0" rpy="0 0 0" />
         <geometry>
-          <mesh filename="package://cob_description/meshes/cob3_torso/head_base_collision.dae" scale="0.01 0.01 0.01"/>
+          <mesh filename="package://cob_description/meshes/cob3_torso/head_base_collision.dae" scale="0.001 0.001 0.001"/>
         </geometry>
       </collision>
