Commit message: tray collision model 10% größer

File: cob_description/urdf/cob3_tray/tray.urdf.xacro (robot description, xacro)
@@ -31,5 +31,5 @@
         <origin xyz="0 0 0" rpy="0 0 0" />
         <geometry>
-          <mesh filename="package://cob_description/meshes/cob3_tray/tray_collision.stl" />
+          <mesh filename="package://cob_description/meshes/cob3_tray/tray_collision.stl" scale="1.1 1.1 1.1"/>
         </geometry>
       </collision>
