Commit message: Neuer Torso

File: cob_description/urdf/cob3_base/base.urdf.xacro (robot description, xacro)
@@ -125,5 +125,5 @@
         <origin xyz="0 0 0" rpy="0 0 0" />
         <geometry>
-          <mesh filename="package://cob_description/meshes/cob3_base/base.stl"/>
+          <mesh filename="package://cob_description/meshes/cob3_base/base_cutted.stl"/>
           <!--box size="${base_size_x} ${base_size_y} ${base_collision_size_z}" /-->
         </geometry>
@@ -133,5 +133,5 @@
         <origin xyz="0 0 0" rpy="0 0 0" />
         <geometry>
-        <mesh filename="package://cob_description/meshes/cob3_base/base_collision.stl"/>
+        <mesh filename="package://cob_description/meshes/cob3_base/base_collision_cutted.stl"/>
           <!--box size="${base_size_x} ${base_size_y} ${base_collision_size_z}" /-->
         </geometry>

Commit message: stl -> dae

File: cob_description/urdf/cob3_base/base.urdf.xacro (robot description, xacro)
@@ -125,5 +125,5 @@
         <origin xyz="0 0 0" rpy="0 0 0" />
         <geometry>
-          <mesh filename="package://cob_description/meshes/cob3_base/base_cutted.stl"/>
+          <mesh filename="package://cob_description/meshes/cob3_base/base_cutted.dae"/>
           <!--box size="${base_size_x} ${base_size_y} ${base_collision_size_z}" /-->
         </geometry>
@@ -133,5 +133,5 @@
         <origin xyz="0 0 0" rpy="0 0 0" />
         <geometry>
-        <mesh filename="package://cob_description/meshes/cob3_base/base_collision_cutted.stl"/>
+        <mesh filename="package://cob_description/meshes/cob3_base/base_collision_cutted.dae"/>
           <!--box size="${base_size_x} ${base_size_y} ${base_collision_size_z}" /-->
         </geometry>

File: cob_description/urdf/cob3_torso/torso_dai.urdf.xacro (robot description, xacro)
@@ -19,5 +19,5 @@
         <origin xyz="0 0 0" rpy="0 0 ${-M_PI/2}" />
         <geometry>
-          <mesh filename="package://cob_description/meshes/cob3_torso/torso_base_high.stl" scale="0.01 0.01 0.01"/>
+          <mesh filename="package://cob_description/meshes/cob3_torso/torso_base_high.dae" scale="0.01 0.01 0.01"/>
         </geometry>
         <material name="IPA/LightGrey" />
@@ -26,5 +26,5 @@
         <origin xyz="0 0 0" rpy="0 0 ${-M_PI/2}" />
         <geometry>
-          <mesh filename="package://cob_description/meshes/cob3_torso/torso_base_low.stl" scale="0.01 0.01 0.01"/>
+          <mesh filename="package://cob_description/meshes/cob3_torso/torso_base_low.dae" scale="0.01 0.01 0.01"/>
         </geometry>
       </collision>
@@ -50,5 +50,5 @@
         <origin xyz="0 -0.055 0" rpy="0 0 0" />
         <geometry>
-          <mesh filename="package://cob_description/meshes/cob3_torso/torso_tilt_high.stl" scale="0.01 0.01 0.01"/>
+          <mesh filename="package://cob_description/meshes/cob3_torso/torso_tilt_high.dae" scale="0.01 0.01 0.01"/>
         </geometry>
         <material name="IPA/LightGrey" />
@@ -57,5 +57,5 @@
         <origin xyz="0 -0.055 0" rpy="0 0 0" />
         <geometry>
-          <mesh filename="package://cob_description/meshes/cob3_torso/torso_tilt_low.stl" scale="0.01 0.01 0.01"/>
+          <mesh filename="package://cob_description/meshes/cob3_torso/torso_tilt_low.dae" scale="0.01 0.01 0.01"/>
         </geometry>
       </collision>
@@ -81,5 +81,5 @@
         <origin xyz="0 0 0" rpy="0 0 0" />
         <geometry>
-          <mesh filename="package://cob_description/meshes/cob3_torso/torso_pan_high.stl" scale="0.01 0.01 0.01"/>
+          <mesh filename="package://cob_description/meshes/cob3_torso/torso_pan_high.dae" scale="0.01 0.01 0.01"/>
         </geometry>
         <material name="IPA/LightGrey" />
@@ -88,5 +88,5 @@
         <origin xyz="0 0 0" rpy="0 0 0" />
         <geometry>
-          <mesh filename="package://cob_description/meshes/cob3_torso/torso_pan_low.stl" scale="0.01 0.01 0.01"/>
+          <mesh filename="package://cob_description/meshes/cob3_torso/torso_pan_low.dae" scale="0.01 0.01 0.01"/>
         </geometry>
       </collision>
@@ -112,5 +112,5 @@
         <origin xyz="0 0 -0.055" rpy="-${M_PI/2} ${M_PI} 0" />
         <geometry>
-          <mesh filename="package://cob_description/meshes/cob3_torso/torso_tilt_high.stl" scale="0.01 0.01 0.01"/>
+          <mesh filename="package://cob_description/meshes/cob3_torso/torso_tilt_high.dae" scale="0.01 0.01 0.01"/>
         </geometry>
         <material name="IPA/LightGrey" />
@@ -120,5 +120,5 @@
         <geometry>
           <!--mesh filename="package://cob_description/meshes/cob3_torso/upper_neck_collision.stl" /-->
-          <mesh filename="package://cob_description/meshes/cob3_torso/torso_tilt_low.stl" scale="0.01 0.01 0.01"/>
+          <mesh filename="package://cob_description/meshes/cob3_torso/torso_tilt_low.dae" scale="0.01 0.01 0.01"/>
         </geometry>
       </collision>
@@ -139,5 +139,5 @@
         <origin xyz="0 0 0" rpy="0 0 0" />
         <geometry>
-          <mesh filename="package://cob_description/meshes/cob3_torso/head_base.stl" scale="0.01 0.01 0.01"/>
+          <mesh filename="package://cob_description/meshes/cob3_torso/head_base.dae" scale="0.01 0.01 0.01"/>
         </geometry>
         <material name="IPA/LightGrey" />
@@ -146,5 +146,5 @@
         <origin xyz="0 0 0" rpy="0 0 0" />
         <geometry>
-          <mesh filename="package://cob_description/meshes/cob3_torso/head_base_collision.stl" scale="0.01 0.01 0.01"/>
+          <mesh filename="package://cob_description/meshes/cob3_torso/head_base_collision.dae" scale="0.01 0.01 0.01"/>
         </geometry>
       </collision>

Commit message: base collision model um 10% größer gemacht

File: cob_description/urdf/cob3_base/base.urdf.xacro (robot description, xacro)
@@ -133,5 +133,5 @@
         <origin xyz="0 0 0" rpy="0 0 0" />
         <geometry>
-        <mesh filename="package://cob_description/meshes/cob3_base/base_collision_cutted.dae"/>
+        <mesh filename="package://cob_description/meshes/cob3_base/base_collision_cutted.dae" scale="1.1 1.1 1.1"/>
           <!--box size="${base_size_x} ${base_size_y} ${base_collision_size_z}" /-->
         </geometry>

Commit message: changes from hydro_dev

File: cob_description/urdf/cob3_base/base.urdf.xacro (robot description, xacro)
@@ -125,5 +125,5 @@
         <origin xyz="0 0 0" rpy="0 0 0" />
         <geometry>
-          <mesh filename="package://cob_description/meshes/cob3_base/base.stl"/>
+          <mesh filename="package://cob_description/meshes/cob3_base/base_cutted.dae"/>
           <!--box size="${base_size_x} ${base_size_y} ${base_collision_size_z}" /-->
         </geometry>
@@ -133,5 +133,5 @@
         <origin xyz="0 0 0" rpy="0 0 0" />
         <geometry>
-        <mesh filename="package://cob_description/meshes/cob3_base/base_collision.stl"/>
+        <mesh filename="package://cob_description/meshes/cob3_base/base_collision_cutted.dae" scale="1.1 1.1 1.1"/>
           <!--box size="${base_size_x} ${base_size_y} ${base_collision_size_z}" /-->
         </geometry>
