Commit message: new asus xtion urdf model

File: cob_description/urdf/cob3_head/head_kinect.urdf.xacro (robot description, xacro)
@@ -3,5 +3,6 @@
   <xacro:include filename="$(find cob_description)/urdf/cob3_head/head.gazebo.xacro" />
   <xacro:include filename="$(find cob_description)/urdf/cob3_head/head.transmission.xacro" />
-  <xacro:include filename="$(find cob_description)/urdf/sensors/kinect.urdf.xacro" />
+  <!--xacro:include filename="$(find cob_description)/urdf/sensors/kinect.urdf.xacro" /-->
+  <xacro:include filename="$(find cob_description)/urdf/sensors/asus_camera.urdf.xacro" />
   <xacro:macro name="head" params="name parent *origin">
     <!-- joint between torso_upper_neck_tilt_link and head_base_link -->
@@ -62,7 +63,13 @@
     </link>
     <!-- cam3d -->
-    <xacro:cob_kinect_v0 name="cam3d" ros_topic="cam3d" parent="${name}_cam_reference_link">
+    <!--xacro:cob_kinect_v0 name="cam3d" ros_topic="cam3d" parent="${name}_cam_reference_link">
       <origin xyz="${cam3d_x} ${cam3d_y} ${cam3d_z}" rpy="${cam3d_roll} ${cam3d_pitch} ${cam3d_yaw}" />
-    </xacro:cob_kinect_v0>
+    </xacro:cob_kinect_v0-->
+    <xacro:asus_camera_model name="cam3d" ros_topic="cam3d" parent="${name}_cam_reference_link">
+      <origin xyz="${cam3d_x} ${cam3d_y} ${cam3d_z}" rpy="${cam3d_roll} ${cam3d_pitch} ${cam3d_yaw}" />
+    </xacro:asus_camera_model>
+    <!--xacro:asus_camera name="cam3d" ros_topic="cam3d" parent="${name}_cam_reference_link">
+      <origin xyz="${cam3d_x} ${cam3d_y} ${cam3d_z}" rpy="${cam3d_roll} ${cam3d_pitch} ${cam3d_yaw}" />
+    </xacro:asus_camera-->
     <!-- extensions -->
     <xacro:head_gazebo name="${name}" />

Commit message: changes from hydro_dev

File: cob_description/urdf/cob3_head/head_kinect.urdf.xacro (robot description, xacro)
@@ -3,5 +3,6 @@
   <xacro:include filename="$(find cob_description)/urdf/cob3_head/head.gazebo.xacro" />
   <xacro:include filename="$(find cob_description)/urdf/cob3_head/head.transmission.xacro" />
-  <xacro:include filename="$(find cob_description)/urdf/sensors/kinect.urdf.xacro" />
+  <!--xacro:include filename="$(find cob_description)/urdf/sensors/kinect.urdf.xacro" /-->
+  <xacro:include filename="$(find cob_description)/urdf/sensors/asus_camera.urdf.xacro" />
   <xacro:macro name="head" params="name parent *origin">
     <!-- joint between torso_upper_neck_tilt_link and head_base_link -->
@@ -73,7 +74,13 @@
     </link>
     <!-- cam3d -->
-    <xacro:cob_kinect_v0 name="cam3d" ros_topic="cam3d" parent="${name}_cam_reference_link">
+    <!--xacro:cob_kinect_v0 name="cam3d" ros_topic="cam3d" parent="${name}_cam_reference_link">
       <origin xyz="${cam3d_x} ${cam3d_y} ${cam3d_z}" rpy="${cam3d_roll} ${cam3d_pitch} ${cam3d_yaw}" />
-    </xacro:cob_kinect_v0>
+    </xacro:cob_kinect_v0-->
+    <xacro:asus_camera_model name="cam3d" ros_topic="cam3d" parent="${name}_cam_reference_link">
+      <origin xyz="${cam3d_x} ${cam3d_y} ${cam3d_z}" rpy="${cam3d_roll} ${cam3d_pitch} ${cam3d_yaw}" />
+    </xacro:asus_camera_model>
+    <!--xacro:asus_camera name="cam3d" ros_topic="cam3d" parent="${name}_cam_reference_link">
+      <origin xyz="${cam3d_x} ${cam3d_y} ${cam3d_z}" rpy="${cam3d_roll} ${cam3d_pitch} ${cam3d_yaw}" />
+    </xacro:asus_camera-->
     <!-- extensions -->
     <xacro:head_gazebo name="${name}" />

File: cob_description/urdf/cob3_tray/tray.urdf.xacro (robot description, xacro)
@@ -27,5 +27,5 @@
         <origin xyz="0 0 0" rpy="0 0 0" />
         <geometry>
-          <mesh filename="package://cob_description/meshes/cob3_tray/tray_collision.stl" />
+          <mesh filename="package://cob_description/meshes/cob3_tray/tray_collision.stl" scale="1.1 1.1 1.1"/>
         </geometry>
       </collision>
